Commit message: Nice Walk

File: Robot/PP/urdf/PP.urdf (robot description, URDF)
Before this commit: robot PP, 13 links, 12 joints
Joints:
- joint LB_ARMPIT: limit lower=-0.6 upper=0.6 effort=1000 velocity=0.5 -> lower=-0.6 upper=0.6 effort=10 velocity=0.188
- joint LB_ELBOW: limit lower=-1 upper=1.2 effort=1000 velocity=0.5 -> lower=-1 upper=1.2 effort=10 velocity=0.188
- joint LB_KNEE: limit lower=-0.6 upper=1.5 effort=1000 velocity=0.5 -> lower=-0.6 upper=1.5 effort=10 velocity=0.188
- joint LF_ARMPIT: limit lower=-0.6 upper=0.6 effort=1000 velocity=0.5 -> lower=-0.6 upper=0.6 effort=10 velocity=0.188
- joint LF_ELBOW: limit lower=-1 upper=1.2 effort=1000 velocity=0.5 -> lower=-1 upper=1.2 effort=10 velocity=0.188
- joint LF_KNEE: limit lower=-0.6 upper=1.5 effort=1000 velocity=0.5 -> lower=-0.6 upper=1.5 effort=10 velocity=0.188
- joint RB_ARMPIT: limit lower=-0.6 upper=0.6 effort=1000 velocity=0.5 -> lower=-0.6 upper=0.6 effort=10 velocity=0.188
- joint RB_ELBOW: limit lower=-1 upper=1.2 effort=1000 velocity=0.5 -> lower=-1 upper=1.2 effort=10 velocity=0.188
- joint RB_KNEE: limit lower=-0.6 upper=1.5 effort=1000 velocity=0.5 -> lower=-0.6 upper=1.5 effort=10 velocity=0.188
- joint RF_ARMPIT: limit lower=-0.6 upper=0.6 effort=1000 velocity=0.5 -> lower=-0.6 upper=0.6 effort=10 velocity=0.188
- joint RF_ELBOW: limit lower=-1 upper=1.2 effort=1000 velocity=0.5 -> lower=-1 upper=1.2 effort=10 velocity=0.188
- joint RF_KNEE: limit lower=-0.6 upper=1.5 effort=1000 velocity=0.5 -> lower=-0.6 upper=1.5 effort=10 velocity=0.188
