Commit message: New URDF & Rob Demo

File: Robot/CML_PP/urdf/CML_PP.urdf (robot description, URDF)
Before this commit: robot CML_PP, 13 links, 12 joints
Links:
- link base_link: geometry collision mesh filename=package://CML_PP/meshes/low_qual/base_link.STL; visual mesh filename=package://CML_PP/meshes/low_qual/base_link.STL
- link lb_calf_link: geometry collision mesh filename=package://CML_PP/meshes/low_qual/lb_calf_link.STL; visual mesh filename=package://CML_PP/meshes/low_qual/lb_calf_link.STL
- link lb_shoulder_link: geometry collision mesh filename=package://CML_PP/meshes/low_qual/lb_shoulder_link.STL; visual mesh filename=package://CML_PP/meshes/low_qual/lb_shoulder_link.STL
- link lb_thigh_link: geometry collision mesh filename=package://CML_PP/meshes/low_qual/lb_thigh_link.STL; visual mesh filename=package://CML_PP/meshes/low_qual/lb_thigh_link.STL
- link lf_calf_link: geometry collision mesh filename=package://CML_PP/meshes/low_qual/lf_calf_link.STL; visual mesh filename=package://CML_PP/meshes/low_qual/lf_calf_link.STL
- link lf_shoulder_link: geometry collision mesh filename=package://CML_PP/meshes/low_qual/lf_shoulder_link.STL; visual mesh filename=package://CML_PP/meshes/low_qual/lf_shoulder_link.STL
- link lf_thigh_link: geometry collision mesh filename=package://CML_PP/meshes/low_qual/lf_thigh_link.STL; visual mesh filename=package://CML_PP/meshes/low_qual/lf_thigh_link.STL
- link rb_calf_link: geometry collision mesh filename=package://CML_PP/meshes/low_qual/rb_calf_link.STL; visual mesh filename=package://CML_PP/meshes/low_qual/rb_calf_link.STL
- link rb_shoulder_link: geometry collision mesh filename=package://CML_PP/meshes/low_qual/rb_shoulder_link.STL; visual mesh filename=package://CML_PP/meshes/low_qual/rb_shoulder_link.STL
- link rb_thigh_link: geometry collision mesh filename=package://CML_PP/meshes/low_qual/rb_thigh_link.STL; visual mesh filename=package://CML_PP/meshes/low_qual/rb_thigh_link.STL
- link rf_calf_link: geometry collision mesh filename=package://CML_PP/meshes/low_qual/rf_calf_link.STL; visual mesh filename=package://CML_PP/meshes/low_qual/rf_calf_link.STL
- link rf_shoulder_link: geometry collision mesh filename=package://CML_PP/meshes/low_qual/rf_shoulder_link.STL; visual mesh filename=package://CML_PP/meshes/low_qual/rf_shoulder_link.STL
- link rf_thigh_link: geometry collision mesh filename=package://CML_PP/meshes/low_qual/rf_thigh_link.STL; visual mesh filename=package://CML_PP/meshes/low_qual/rf_thigh_link.STL
