Commit message: WALK test with parameters in accurate simulation 1

File: CML/Simulation Control/PinkPanther_CML/urdf/pp_urdf_final.urdf (robot description, URDF)
Before this commit: robot PinkPanther_CML, 13 links, 12 joints
Joints:
- joint lb_elbow_joint: limit lower=-0.6 upper=1.2 effort=1.667 velocity=6.545 -> lower=-0.9 upper=1.2 effort=1.667 velocity=6.545
